File: Speed Control Fan.kicad_sch (KiCad schematic)
At the start: 11 parts

Commit message: Add files via upload
Parts:
- added D?: RB205T-60NZC9, TO254P480X1010X2100-3P, symbol LibraryLoader:RB205T-60NZC9
- added F?: Fuse, symbol Device:Fuse
- added J?: Conn_01x04_Male, symbol Connector:Conn_01x04_Male
- added J? (x2): Conn_01x02_Male, symbol Connector:Conn_01x02_Male
- added Q?: IXTP60N20X4, TO254P470X1000X2010-3P, symbol LibraryLoader:IXTP60N20X4
- added R? (x2): R, symbol Device:R
- R? (x4): value 2k -> 1k
- R?: value 10k -> 36k
- R?: value 24k -> 10k
Connections:
- net V_Out: now reaches J?.1 (Pin_1), J?.1 (Pin_1), J?.1 (Pin_1), J?.1 (Pin_1), R?.2, U?.3
- net 48V Line renamed 24V Line
- net 24V Line: now also D?.1 (A_1), J?.1 (Pin_1), J?.1 (Pin_1)
- net microcontroller/GND renamed GND
- net GND: now also J?.2 (Pin_2), J?.4 (Pin_4), Q?.3, R?.2
- net microcontroller/PA10 renamed Tach4
- net microcontroller/PA14 renamed PWM1
- net microcontroller/PA4: no longer names the net of R?.2
- net microcontroller/PA8 renamed Tach2
- net microcontroller/PA9 renamed Tach3
- net microcontroller/PB0 renamed PWM2
- net microcontroller/PB1 renamed PWM3
- net microcontroller/PB2 renamed PWM4
- new net: F?.1, J?.3 (Pin_3)
- new net: Q?.1, R?.2
- new net: D?.2 (K), J?.2 (Pin_2), Q?.2
- new net +24V: F?.2
- new net Can1H: J?.1 (Pin_1)
- new net Can1L: J?.2 (Pin_2)
- new net WaterPumpPwm: R?.1, R?.1
Other:
- removed sheet StandardizedVRMS
- added sheet VRMS (../../2023KicadLibrary/Standardized Subsheets/vrmsv2.kicad_sch)
- note added: "PumpMoter"
- moved on the sheet: J?, R?

Commit message: Add files via upload
Parts:
- removed D?: RB205T-60NZC9, TO254P480X1010X2100-3P, symbol LibraryLoader:RB205T-60NZC9
- removed F?: Fuse, symbol Device:Fuse
- removed J?: Conn_01x04_Male, symbol Connector:Conn_01x04_Male
- removed J? (x2): Conn_01x02_Male, symbol Connector:Conn_01x02_Male
- removed Q?: IXTP60N20X4, TO254P470X1000X2010-3P, symbol LibraryLoader:IXTP60N20X4
- removed R? (x2): R, symbol Device:R
- R? (x4): value 1k -> 2k
- R?: value 36k -> 10k
- R?: value 10k -> 24k
Connections:
- net microcontroller/PA4: now reaches R?.2
- net 24V Line renamed 48V Line
- net GND renamed microcontroller/GND
- net PWM1 renamed microcontroller/PA14
- net PWM2 renamed microcontroller/PB0
- net PWM3 renamed microcontroller/PB1
- net PWM4 renamed microcontroller/PB2
- net Tach2 renamed microcontroller/PA8
- net Tach3 renamed microcontroller/PA9
- net Tach4 renamed microcontroller/PA10
- net V_Out: no longer names the net of J?.1 (Pin_1), J?.1 (Pin_1), J?.1 (Pin_1), J?.1 (Pin_1), R?.2, U?.3
Other:
- removed sheet VRMS
- added sheet StandardizedVRMS (Standardized Subsheets/StandardizedVRMS.kicad_sch)
- note removed: "PumpMoter"
- moved on the sheet: J?, R?

Commit message: Initial commit (?)
Parts:
- removed J? (x4): Conn_01x04_Male, symbol Connector:Conn_01x04_Male
- removed R? (x4): 2k, symbol Device:R
- removed R?: 10k, symbol Device:R
- removed R?: 24k, symbol Device:R
- added F?: Fuse, symbol Device:Fuse
- added J?: Conn_01x04_Male, symbol Connector:Conn_01x04_Male
Connections:
- net microcontroller/PA3: now also U?.1 (+)
- net VOUT: now reaches U?.3
- net 48V Line renamed +24V
- net +24V: now also F?.2
- net microcontroller/GND renamed GND
- net GND: now also J?.4 (Pin_4)
- new net: F?.1, J?.3 (Pin_3)
- new net Can1H: J?.1 (Pin_1)
- new net Can1L: J?.2 (Pin_2)
Other:
- removed sheet StandardizedVRMS
- added sheet Fans (Fans.kicad_sch)
- added sheet VRMS (../../2023KicadLibrary/Standardized Subsheets/vrmsv2.kicad_sch)
- added sheet WaterPump (WaterPump.kicad_sch)

Commit message: message
Parts:
- removed U?: OPAMP, symbol pspice:OPAMP
- added Q?: IXTP60N20X4, TO254P470X1000X2010-3P, symbol LibraryLoader:IXTP60N20X4
- added R?: R, symbol Device:R
Connections:
- net +24V: now also R?.1
- net GND: now also Q?.3
- net VOUT: now also Q?.2, R?.2
- net microcontroller/PA3: now also Q?.1
Other:
- added sheet Matt's Cooling Disable (Cooling_Disable.kicad_sch)
